File: lin_bluetooth_gateway/lin_bluetooth_gateway.sch (KiCad schematic (older format))
At the start: 9 parts, among them P1 CONN_01X01, P2 CONN_01X01, P3 CONN_01X01, P4 CONN_01X03, U1 MCP2050, U2 BL652

Commit message: lin_bluetooth_gateway rev2
Parts:
- removed P1, P2, P3: CONN_01X01, Wire_Pads:SolderWirePad_single_1-2mmDrill, symbol CONN_01X01
- added P1, P2: MOLEX-0431603103, Connectors_Molex:Molex_Sabre_43160-XX03_03x7.49mm_Angled_BoardLock, symbol CONN_01X03
- added R1: 10k, Resistors_SMD:R_0603_HandSoldering, symbol R
Connections:
- net labels added: 12V_UNPROTECTED, CS/LWAKE, FAULT, RXD, TXD, VBAT_RATIO
- wire segments 25 -> 39
- no-connect marks 32 -> 31
Other:
- moved on the sheet: D1, D2, P4, R2, U1, U2

Commit message: minor updates (DigiKey PN, cleaning)
Parts:
- D2: value D -> 1N4148
- P4: DIGIKEY (none) -> 952-1351-5-ND
- R1, R2: DIGIKEY (none) -> 311-10KGRCT-ND
- U1: DIGIKEY (none) -> MCP2050-330E/SL-ND
- U2: DIGIKEY (none) -> BL652-SA-01-CT-ND
Changed lines of the file:
@@
 F 2 "footprints:BL652-SA" H 5550 4250 60  0001 C CNN
 F 3 "" H 5550 4250 60  0001 C CNN
+F 4 "BL652-SA-01-CT-ND" H 5300 5650 60  0000 C CNN "DIGIKEY"
 	1    5550 4250
 	1    0    0    -1
@@
 F 2 "Housings_SOIC:SOIC-14_3.9x8.7mm_Pitch1.27mm" H 4900 1900 60  0001 C CNN
 F 3 "http://ww1.microchip.com/downloads/en/DeviceDoc/22299B.pdf" H 4900 1900 60  0001 C CNN
+F 4 "MCP2050-330E/SL-ND" H 5350 2550 60  0000 C CNN "DIGIKEY"
 	1    5350 1850
 	1    0    0    -1
@@
 F 2 "Resistors_SMD:R_0603_HandSoldering" V 6980 1750 50  0001 C CNN
 F 3 "" H 7050 1750 50  0000 C CNN
+F 4 "311-10KGRCT-ND" V 7200 1750 60  0000 C CNN "DIGIKEY"
 	1    7050 1750
 	1    0    0    -1
@@
 L PWR_FLAG #FLG04
 U 1 1 58074312
-P 3000 1250
-F 0 "#FLG04" H 3000 1345 50  0001 C CNN
-F 1 "PWR_FLAG" H 3000 1430 50  0000 C CNN
-F 2 "" H 3000 1250 50  0000 C CNN
-F 3 "" H 3000 1250 50  0000 C CNN
-	1    3000 1250
+P 3750 1250
+F 0 "#FLG04" H 3750 1345 50  0001 C CNN
+F 1 "PWR_FLAG" H 3750 1430 50  0000 C CNN
+F 2 "" H 3750 1250 50  0000 C CNN
+F 3 "" H 3750 1250 50  0000 C CNN
+	1    3750 1250
 	1    0    0    -1
 $EndComp
@@
 F 2 "Pin_Headers:Pin_Header_Straight_1x04_Pitch2.00mm" H 4000 4750 50  0001 C CNN
 F 3 "" H 4000 4750 50  0000 C CNN
+F 4 "952-1351-5-ND" V 4200 4750 60  0000 C CNN "DIGIKEY"
 	1    4000 4750
 	-1   0    0    -1
@@
 P 3400 1450
 F 0 "D2" H 3400 1550 50  0000 C CNN
-F 1 "D" H 3400 1350 50  0000 C CNN
+F 1 "1N4148" H 3400 1350 50  0000 C CNN
 F 2 "Diodes_SMD:SOD-123" H 3400 1450 50  0001 C CNN
 F 3 "http://www.diodes.com/_files/datasheets/ds30086.pdf" H 3400 1450 50  0001 C CNN
-F 4 "1N4148W-FDICT-ND" H 3400 1450 60  0001 C CNN "DIGIKEY"
+F 4 "1N4148W-FDICT-ND" H 3550 1250 60  0000 C CNN "DIGIKEY"
 	1    3400 1450
 	-1   0    0    1
@@
 P 3750 2150
 F 0 "D1" H 3750 2250 50  0000 C CNN
-F 1 "RSB36V" H 3750 2050 50  0000 C CNN
+F 1 "RSB36V" V 3700 1950 50  0000 C CNN
 F 2 "Diodes_SMD:SOD-323_HandSoldering" H 3750 2150 50  0001 C CNN
 F 3 "http://rohmfs.rohm.com/en/products/databook/datasheet/discrete/diode/zener/rsb36v.pdf" H 3750 2150 50  0001 C CNN
-F 4 "RSB36VTE-17CT-ND" H 3750 2150 60  0001 C CNN "DIGIKEY"
+F 4 "RSB36VTE-17CT-ND" V 3800 1600 60  0000 C CNN "DIGIKEY"
 	1    3750 2150
 	0    1    1    0
@@
 U 1 1 583D2468
 P 3750 1750
-F 0 "R1" V 3830 1750 50  0000 C CNN
+F 0 "R1" H 3650 1800 50  0000 C CNN
 F 1 "10k" V 3750 1750 50  0000 C CNN
 F 2 "Resistors_SMD:R_0603_HandSoldering" V 3680 1750 50  0001 C CNN
 F 3 "" H 3750 1750 50  0000 C CNN
+F 4 "311-10KGRCT-ND" H 3250 1700 60  0000 C CNN "DIGIKEY"
 	1    3750 1750
 	1    0    0    -1
 $EndComp
 Wire Wire Line
-	3750 1450 3750 1600
+	3750 1250 3750 1600
 $Comp
 L CONN_01X03 P1
@@
 F 2 "Connectors_Molex:Molex_Sabre_43160-XX03_03x7.49mm_Angled_BoardLock" H 2350 1150 50  0001 C CNN
 F 3 "http://www.molex.com/pdm_docs/sd/431603103_sd.pdf" H 2350 1150 50  0001 C CNN
-F 4 "WM18489-ND" H 2350 1150 60  0001 C CNN "DIGIKEY"
+F 4 "WM18489-ND" V 2550 1150 60  0000 C CNN "DIGIKEY"
 	1    2350 1150
 	0    1    -1   0
@@
 	1500 1450 3250 1450
 Connection ~ 3750 1450
-Connection ~ 3000 1450
 Wire Wire Line
 	3750 2250 3750 2350
@@
 F 2 "Connectors_Molex:Molex_Sabre_43160-XX03_03x7.49mm_Angled_BoardLock" H 1400 1150 50  0001 C CNN
 F 3 "http://www.molex.com/pdm_docs/sd/431603103_sd.pdf" H 1400 1150 50  0001 C CNN
-F 4 "WM18489-ND" H 1400 1150 60  0001 C CNN "DIGIKEY"
+F 4 "WM18489-ND" V 1600 1150 60  0000 C CNN "DIGIKEY"
 	1    1400 1150
 	0    1    -1   0
@@
 	2450 1350 2450 1450
 Wire Wire Line
-	3000 1250 3000 1450
-Wire Wire Line
 	2350 1350 2350 1950
