File: 13a_switch_x4/kicad/13a_switch_x4.kicad_pcb (KiCad board)
At the start: 2 copper layers, 87.6 x 41.9 mm, 27 parts, among them P1 MOLEX-0431603103, P2 MOLEX-0431603103, P3 MOLEX-22-28-6050, P4 TE-282836-4, P5 TE-282836-4, Q1 Q_NMOS_GDSD, Q2 Q_NMOS_GDSD, Q3 Q_NMOS_GDSD, Q4 Q_NMOS_GDSD, U1 PIC16F1829LIN

Commit message: Using SW_DIP_x04 from KiCad library
Parts:
- removed S1: DIP_SWITCH_4, footprints:Copal_CHS-04TB
- added SW1: SW_DIP_x04, Buttons_Switches_SMD:SW_SPST_Copal_CHS-04TB, F.Cu at (136.5, 81.3)
Changed lines of the file:
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@@
   (page A4)
   (layers
-    (0 F.Cu signal hide)
-    (31 B.Cu signal hide)
+    (0 F.Cu signal)
+    (31 B.Cu signal)
     (32 B.Adhes user)
     (33 F.Adhes user)
@@
     (aux_axis_origin 0 0)
     (grid_origin 146.685 57.785)
-    (visible_elements FFFEEF7F)
+    (visible_elements FFFEFF7F)
     (pcbplotparams
       (layerselection 0x00030_80000001)
@@
     )
   )
-  (module footprints:Copal_CHS-04TB (layer F.Cu)
+  (module Mounting_Holes:MountingHole_2.7mm_Pad_Via (layer F.Cu)
+    (at 107.315 52.07)
+    (descr "Mounting Hole 2.7mm")
+    (tags "mounting hole 2.7mm")
+    (fp_text reference REF** (at 0 -3.7) (layer F.SilkS) hide
+      (effects (font (size 1 1) (thickness 0.15)))
+    )
+    (fp_text value MountingHole_2.7mm_Pad_Via (at 0 3.7) (layer F.Fab)
+      (effects (font (size 1 1) (thickness 0.15)))
+    )
+    (fp_circle (center 0 0) (end 2.7 0) (layer Cmts.User) (width 0.15))
+    (fp_circle (center 0 0) (end 2.95 0) (layer F.CrtYd) (width 0.05))
+    (pad 1 thru_hole circle (at 0 0) (size 5.4 5.4) (drill 2.7) (layers *.Cu *.Mask))
+    (pad "" thru_hole circle (at 2.025 0) (size 0.6 0.6) (drill 0.5) (layers *.Cu *.Mask))
+    (pad "" thru_hole circle (at 1.431891 1.431891) (size 0.6 0.6) (drill 0.5) (layers *.Cu *.Mask))
+    (pad "" thru_hole circle (at 0 2.025) (size 0.6 0.6) (drill 0.5) (layers *.Cu *.Mask))
+    (pad "" thru_hole circle (at -1.431891 1.431891) (size 0.6 0.6) (drill 0.5) (layers *.Cu *.Mask))
+    (pad "" thru_hole circle (at -2.025 0) (size 0.6 0.6) (drill 0.5) (layers *.Cu *.Mask))
+    (pad "" thru_hole circle (at -1.431891 -1.431891) (size 0.6 0.6) (drill 0.5) (layers *.Cu *.Mask))
+    (pad "" thru_hole circle (at 0 -2.025) (size 0.6 0.6) (drill 0.5) (layers *.Cu *.Mask))
+    (pad "" thru_hole circle (at 1.431891 -1.431891) (size 0.6 0.6) (drill 0.5) (layers *.Cu *.Mask))
+  )
+  (module Buttons_Switches_SMD:SW_SPST_Copal_CHS-04TB (layer F.Cu)
     (at 136.525 81.28 180)
     (descr "8-Lead Plastic Small Outline (SM) - Medium, 5.28 mm Body [SOIC] (see Microchip Packaging Specification 00000049BS.pdf)")
     (tags "SOIC 1.27")
     (attr smd)
-    (fp_text reference S1 (at 0 -4.191 180) (layer F.SilkS)
-      (effects (font (size 1 1) (thickness 0.15)))
-    )
-    (fp_text value DIP_SWITCH_4 (at 0 4.318 180) (layer F.Fab)
+    (fp_text reference SW1 (at 0 -4.191 180) (layer F.SilkS)
+      (effects (font (size 1 1) (thickness 0.15)))
+    )
+    (fp_text value SW_DIP_x04 (at 0 4.318 180) (layer F.Fab)
       (effects (font (size 1 1) (thickness 0.15)))
     )
@@
     (pad 1 smd rect (at -3.65 -1.905 180) (size 1.7 0.65) (layers F.Cu F.Paste F.Mask)
       (net 22 /A0))
-    (pad 3 smd rect (at -3.65 -0.635 180) (size 1.7 0.65) (layers F.Cu F.Paste F.Mask)
+    (pad 2 smd rect (at -3.65 -0.635 180) (size 1.7 0.65) (layers F.Cu F.Paste F.Mask)
       (net 23 /A1))
-    (pad 5 smd rect (at -3.65 0.635 180) (size 1.7 0.65) (layers F.Cu F.Paste F.Mask)
+    (pad 3 smd rect (at -3.65 0.635 180) (size 1.7 0.65) (layers F.Cu F.Paste F.Mask)
       (net 24 /A2))
-    (pad 7 smd rect (at -3.65 1.905 180) (size 1.7 0.65) (layers F.Cu F.Paste F.Mask)
+    (pad 4 smd rect (at -3.65 1.905 180) (size 1.7 0.65) (layers F.Cu F.Paste F.Mask)
       (net 25 /A3))
-    (pad 8 smd rect (at 3.65 1.905 180) (size 1.7 0.65) (layers F.Cu F.Paste F.Mask)
+    (pad 5 smd rect (at 3.65 1.905 180) (size 1.7 0.65) (layers F.Cu F.Paste F.Mask)
       (net 2 GND))
     (pad 6 smd rect (at 3.65 0.635 180) (size 1.7 0.65) (layers F.Cu F.Paste F.Mask)
       (net 2 GND))
-    (pad 4 smd rect (at 3.65 -0.635 180) (size 1.7 0.65) (layers F.Cu F.Paste F.Mask)
-      (net 2 GND))
-    (pad 2 smd rect (at 3.65 -1.905 180) (size 1.7 0.65) (layers F.Cu F.Paste F.Mask)
-      (net 2 GND))
-    (model /home/cpriscal/projects/fluffy-potato/common/kicad/copal-chs-04tb.wrl
-      (at (xyz 0 0 0))
-      (scale (xyz 1 1 1))
-      (rotate (xyz 0 0 0))
-    )
-  )
-  (module Mounting_Holes:MountingHole_2.7mm_Pad_Via (layer F.Cu)
-    (at 107.315 52.07)
-    (descr "Mounting Hole 2.7mm")
-    (tags "mounting hole 2.7mm")
-    (fp_text reference REF** (at 0 -3.7) (layer F.SilkS) hide
-      (effects (font (size 1 1) (thickness 0.15)))
-    )
-    (fp_text value MountingHole_2.7mm_Pad_Via (at 0 3.7) (layer F.Fab)
-      (effects (font (size 1 1) (thickness 0.15)))
-    )
-    (fp_circle (center 0 0) (end 2.7 0) (layer Cmts.User) (width 0.15))
-    (fp_circle (center 0 0) (end 2.95 0) (layer F.CrtYd) (width 0.05))
-    (pad 1 thru_hole circle (at 0 0) (size 5.4 5.4) (drill 2.7) (layers *.Cu *.Mask))
-    (pad "" thru_hole circle (at 2.025 0) (size 0.6 0.6) (drill 0.5) (layers *.Cu *.Mask))
-    (pad "" thru_hole circle (at 1.431891 1.431891) (size 0.6 0.6) (drill 0.5) (layers *.Cu *.Mask))
-    (pad "" thru_hole circle (at 0 2.025) (size 0.6 0.6) (drill 0.5) (layers *.Cu *.Mask))
-    (pad "" thru_hole circle (at -1.431891 1.431891) (size 0.6 0.6) (drill 0.5) (layers *.Cu *.Mask))
-    (pad "" thru_hole circle (at -2.025 0) (size 0.6 0.6) (drill 0.5) (layers *.Cu *.Mask))
-    (pad "" thru_hole circle (at -1.431891 -1.431891) (size 0.6 0.6) (drill 0.5) (layers *.Cu *.Mask))
-    (pad "" thru_hole circle (at 0 -2.025) (size 0.6 0.6) (drill 0.5) (layers *.Cu *.Mask))
-    (pad "" thru_hole circle (at 1.431891 -1.431891) (size 0.6 0.6) (drill 0.5) (layers *.Cu *.Mask))
+    (pad 7 smd rect (at 3.65 -0.635 180) (size 1.7 0.65) (layers F.Cu F.Paste F.Mask)
+      (net 2 GND))
+    (pad 8 smd rect (at 3.65 -1.905 180) (size 1.7 0.65) (layers F.Cu F.Paste F.Mask)
+      (net 2 GND))
+    (model Buttons_Switches_SMD.3dshapes/SW_SPST_Copal_CHS-04TB.wrl
+      (at (xyz 0 0 0))
+      (scale (xyz 1 1 1))
+      (rotate (xyz 0 0 0))
+    )
   )
   (gr_text "2016 Cedric Priscal" (at 123.825 88.9) (layer F.SilkS)

Commit message: [13a_switch_x4] Using official libraries
Parts:
- SW1: footprint Buttons_Switches_SMD:SW_SPST_Copal_CHS-04TB -> Buttons_Switches_SMD:SW_DIP_x4_W7.62mm_Slide_Copal_CHS-B
