File: 13a_switch_x4/kicad/13a_switch_x4.sch (KiCad schematic (older format))
At the start: 23 parts, among them P1 MOLEX-0431603103, P2 MOLEX-0431603103, P3 MOLEX-22-28-6050, P4 TE-282836-4, P5 TE-282836-4, Q1 Q_NMOS_GDSD, Q2 Q_NMOS_GDSD, Q3 Q_NMOS_GDSD, Q4 Q_NMOS_GDSD, U1 PIC16F1829LIN

Commit message: Moving PIC16F1829LIN symbol to microchip library
Parts:
- D3, D4, D5, D6: symbol LED -> LED-RESCUE-13a_switch_x4
Other:
- moved on the sheet: U1

Commit message: Using SW_DIP_x04 from KiCad library
Parts:
- removed S1: DIP_SWITCH_4, footprints:Copal_CHS-04TB, symbol DIP_SWITCH_4
- added SW1: SW_DIP_x04, Buttons_Switches_SMD:SW_SPST_Copal_CHS-04TB, symbol SW_DIP_x04
Changed lines of the file:
@@
 LIBS:valves
 LIBS:fluffy-potato
+LIBS:switches
 LIBS:13a_switch_x4-cache
 EELAYER 25 0
@@
 F 3 "" H 3550 7100 50  0000 C CNN
 	1    3550 7100
-	1    0    0    -1
-$EndComp
-$Comp
-L DIP_SWITCH_4 S1
-U 1 1 5844A01A
-P 3200 6700
-F 0 "S1" H 3200 7000 60  0000 C CNN
-F 1 "DIP_SWITCH_4" H 3200 6400 60  0000 C CNN
-F 2 "footprints:Copal_CHS-04TB" H 3250 7050 60  0001 C CNN
-F 3 "http://www.nidec-copal-electronics.com/e/catalog/switch/chs.pdf" H 3250 7050 60  0001 C CNN
-F 4 "563-1008-1-ND" H 3200 7100 60  0000 C CNN "DIGIKEY"
-	1    3200 6700
 	1    0    0    -1
 $EndComp
@@
 	6000 6300 6000 6400
 Connection ~ 6000 6400
+$Comp
+L SW_DIP_x04 SW1
+U 1 1 5862DCE9
+P 3200 6750
+F 0 "SW1" H 3200 7100 50  0000 C CNN
+F 1 "SW_DIP_x04" H 3200 6500 50  0000 C CNN
+F 2 "Buttons_Switches_SMD:SW_SPST_Copal_CHS-04TB" H 3200 6750 50  0001 C CNN
+F 3 "" H 3200 6750 50  0000 C CNN
+F 4 "563-1008-1-ND" V 2600 6750 60  0000 C CNN "DIGIKEY"
+	1    3200 6750
+	1    0    0    -1
+$EndComp
 $EndSCHEMATC

Commit message: [13a_switch_x4] Using official libraries
Parts:
- SW1: footprint Buttons_Switches_SMD:SW_SPST_Copal_CHS-04TB -> Buttons_Switches_SMD:SW_DIP_x4_W7.62mm_Slide_Copal_CHS-B
Changed lines of the file:
@@
 EESchema Schematic File Version 2
+LIBS:13a_switch_x4-rescue
 LIBS:power
 LIBS:device
@@
 LIBS:contrib
 LIBS:valves
-LIBS:fluffy-potato
 LIBS:switches
+LIBS:microchip_pic16mcu
 LIBS:13a_switch_x4-cache
 EELAYER 25 0
@@
 L +12V #PWR01
 U 1 1 57DF768A
-P 4250 1850
-F 0 "#PWR01" H 4250 1700 50  0001 C CNN
-F 1 "+12V" H 4250 1990 50  0000 C CNN
-F 2 "" H 4250 1850 50  0000 C CNN
-F 3 "" H 4250 1850 50  0000 C CNN
-	1    4250 1850
-	1    0    0    -1
-$EndComp
-Text Label 2900 3250 0    60   ~ 0
+P 4350 2350
+F 0 "#PWR01" H 4350 2200 50  0001 C CNN
+F 1 "+12V" H 4350 2490 50  0000 C CNN
+F 2 "" H 4350 2350 50  0000 C CNN
+F 3 "" H 4350 2350 50  0000 C CNN
+	1    4350 2350
+	1    0    0    -1
+$EndComp
+Text Label 2950 3300 0    60   ~ 0
 /MCLR
-Text Label 2900 2850 0    60   ~ 0
+Text Label 2950 3000 0    60   ~ 0
 ICSPDAT
-Text Label 2900 3050 0    60   ~ 0
+Text Label 2950 3100 0    60   ~ 0
 ICSPCLK
 $Comp
@@
 L GND #PWR03
 U 1 1 57DFB653
-P 4550 5100
-F 0 "#PWR03" H 4550 4850 50  0001 C CNN
-F 1 "GND" H 4550 4950 50  0000 C CNN
-F 2 "" H 4550 5100 50  0000 C CNN
-F 3 "" H 4550 5100 50  0000 C CNN
-	1    4550 5100
+P 4550 4600
+F 0 "#PWR03" H 4550 4350 50  0001 C CNN
+F 1 "GND" H 4550 4450 50  0000 C CNN
+F 2 "" H 4550 4600 50  0000 C CNN
+F 3 "" H 4550 4600 50  0000 C CNN
+	1    4550 4600
 	1    0    0    -1
 $EndComp
@@
 L +5V #PWR05
 U 1 1 57DFC341
-P 4550 1850
-F 0 "#PWR05" H 4550 1700 50  0001 C CNN
-F 1 "+5V" H 4550 1990 50  0000 C CNN
-F 2 "" H 4550 1850 50  0000 C CNN
-F 3 "" H 4550 1850 50  0000 C CNN
-	1    4550 1850
+P 4500 2350
+F 0 "#PWR05" H 4500 2200 50  0001 C CNN
+F 1 "+5V" H 4500 2490 50  0000 C CNN
+F 2 "" H 4500 2350 50  0000 C CNN
+F 3 "" H 4500 2350 50  0000 C CNN
+	1    4500 2350
 	1    0    0    -1
 $EndComp
@@
 	1    0    0    -1
 $EndComp
-Text Label 2950 3750 0    60   ~ 0
+Text Label 2950 3900 0    60   ~ 0
 LBUS
 Text Label 8950 1100 0    60   ~ 0
@@
 P 4450 3500
 F 0 "U1" H 4500 3600 60  0000 C CNN
-F 1 "PIC16F1829LIN" H 5400 2150 60  0000 C CNN
+F 1 "PIC16F1829LIN" H 4500 3450 60  0000 C CNN
 F 2 "Housings_SSOP:SSOP-20_5.3x7.2mm_Pitch0.65mm" H 4450 3500 60  0001 C CNN
 F 3 "http://ww1.microchip.com/downloads/en/DeviceDoc/41673A.pdf" H 4450 3500 60  0001 C CNN
-F 4 "PIC16F1829LIN-I/SS-ND" H 5400 2050 60  0000 C CNN "DIGIKEY"
+F 4 "PIC16F1829LIN-I/SS-ND" H 5300 4450 60  0000 C CNN "DIGIKEY"
 	1    4450 3500
 	1    0    0    -1
@@
 Text Label 2800 6850 2    60   ~ 0
 A3
-Text Label 5500 2700 0    60   ~ 0
+Text Label 3550 3200 2    60   ~ 0
 A0
-Text Label 5500 3300 0    60   ~ 0
+Text Label 5350 3800 0    60   ~ 0
 A1
-Text Label 5500 3500 0    60   ~ 0
+Text Label 5350 3700 0    60   ~ 0
 A2
-Text Label 5500 3700 0    60   ~ 0
+Text Label 5350 3600 0    60   ~ 0
 A3
-Text Label 5500 2900 0    60   ~ 0
+Text Label 3550 3400 2    60   ~ 0
 CMD_1
-Text Label 5500 4300 0    60   ~ 0
+Text Label 5350 3300 0    60   ~ 0
 CMD_2
-Text Label 5500 3900 0    60   ~ 0
+Text Label 5350 3500 0    60   ~ 0
 CMD_3
-Text Label 5500 4100 0    60   ~ 0
+Text Label 5350 3400 0    60   ~ 0
 CMD_4
-NoConn ~ 5500 3100
-Wire Wire Line
-	2800 3250 3400 3250
-Wire Wire Line
-	2800 2850 3400 2850
-Wire Wire Line
-	2800 3050 3400 3050
+NoConn ~ 3550 3500
+Wire Wire Line
+	2950 3300 3550 3300
+Wire Wire Line
+	2950 3000 3550 3000
+Wire Wire Line
+	2950 3100 3550 3100
 Wire Wire Line
 	8300 1750 8300 1750
@@
 	7900 1550 8000 1550
 Wire Wire Line
-	3400 3950 3250 3950
-Wire Wire Line
-	3250 3950 3250 4150
-Wire Wire Line
-	3250 4150 3400 4150
-Wire Wire Line
-	4350 4900 4350 5000
-Wire Wire Line
-	4550 4900 4550 5100
-Wire Wire Line
-	4250 1850 4250 2100
-Wire Wire Line
-	2750 3750 3400 3750
-Wire Wire Line
-	4450 2100 4450 1950
-Wire Wire Line
-	4450 1950 4650 1950
-Wire Wire Line
-	4650 1950 4650 2100
-Wire Wire Line
-	4550 1950 4550 1850
-Connection ~ 4550 1950
+	3550 3700 3450 3700
+Wire Wire Line
+	3450 3700 3450 3800
+Wire Wire Line
+	3450 3800 3550 3800
+Wire Wire Line
+	4350 4400 4350 4500
+Wire Wire Line
+	4550 4400 4550 4600
+Wire Wire Line
+	4350 2350 4350 2600
+Wire Wire Line
+	2750 3900 3550 3900
+Wire Wire Line
+	4450 2600 4450 2450
+Wire Wire Line
+	4450 2450 4550 2450
+Wire Wire Line
+	4550 2450 4550 2600
+Wire Wire Line
+	4500 2450 4500 2350
+Connection ~ 4500 2450
 Wire Wire Line
 	8300 1350 8300 1100
 Wire Wire Line
-	2750 4200 2750 3750
+	2750 4200 2750 3900
 Wire Wire Line
 	1900 2800 1350 2800
@@
 	1250 2900 1250 2850
 Wire Wire Line
-	4350 5000 4550 5000
-Connection ~ 4550 5000
+	4350 4500 4550 4500
+Connection ~ 4550 4500
 Wire Wire Line
 	2750 4600 2750 5000
@@
 F 0 "SW1" H 3200 7100 50  0000 C CNN
 F 1 "SW_DIP_x04" H 3200 6500 50  0000 C CNN
-F 2 "Buttons_Switches_SMD:SW_SPST_Copal_CHS-04TB" H 3200 6750 50  0001 C CNN
+F 2 "Buttons_Switches_SMD:SW_DIP_x4_W7.62mm_Slide_Copal_CHS-B" H 3200 6750 50  0001 C CNN
 F 3 "" H 3200 6750 50  0000 C CNN
 F 4 "563-1008-1-ND" V 2600 6750 60  0000 C CNN "DIGIKEY"
