File: edge-connector-motherboard/edge-connector-motherboard.kicad_pcb (KiCad board)
At the start: 2 copper layers, 35.6 x 132.1 mm, 21 parts, among them J1 Screw_Terminal_1x01, J10 Screw_Terminal_1x01, J11 Screw_Terminal_1x01, J12 Screw_Terminal_1x01, J13 Screw_Terminal_1x01, J14 Screw_Terminal_1x01, J15 Screw_Terminal_1x01, J2 Screw_Terminal_1x01, J3 Screw_Terminal_1x01, J4 Screw_Terminal_1x01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

Commit message: edge-connector-motherboard: adding 3d models and digikey references
Routing:
- net GNDPWR: track 221.2 -> 200.9 mm
- net GND: track 87.3 -> 107.6 mm
Changed lines of the file:
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@@
   (general
     (links 126)
-    (no_connects 3)
+    (no_connects 5)
     (area 126.924999 29.134999 162.635001 161.365001)
     (thickness 1.6)
@@
     (pad 1 thru_hole circle (at -2.5 3.5) (size 3 3) (drill 1.85) (layers *.Cu *.Mask)
       (net 1 +12V))
+    (model ../../../../../home/cpriscal/Projets/fluffy-potato/edge-connector-motherboard/keystone-PN7770.wrl
+      (at (xyz 0.155 0 -0.2))
+      (scale (xyz 0.393701 0.393701 0.393701))
+      (rotate (xyz -90 0 90))
+    )
   )
   (module edge-connector-motherboard:TERM_SCREW_M3 (layer F.Cu)
@@
     (pad 1 thru_hole circle (at -2.5 3.5) (size 3 3) (drill 1.85) (layers *.Cu *.Mask)
       (net 4 /PIC16F1829LIN/LBUS))
+    (model ../../../../../home/cpriscal/Projets/fluffy-potato/edge-connector-motherboard/keystone-PN7770.wrl
+      (at (xyz 0.155 0 -0.2))
+      (scale (xyz 0.393701 0.393701 0.393701))
+      (rotate (xyz -90 0 90))
+    )
   )
   (module edge-connector-motherboard:TERM_SCREW_M3 (layer F.Cu)
@@
     (pad 1 thru_hole circle (at -2.5 3.5) (size 3 3) (drill 1.85) (layers *.Cu *.Mask)
       (net 26 GNDPWR))
+    (model ../../../../../home/cpriscal/Projets/fluffy-potato/edge-connector-motherboard/keystone-PN7770.wrl
+      (at (xyz 0.155 0 -0.2))
+      (scale (xyz 0.393701 0.393701 0.393701))
+      (rotate (xyz -90 0 90))
+    )
   )
   (module edge-connector-motherboard:TERM_SCREW_M3 (layer F.Cu)
@@
     (pad 1 thru_hole circle (at -2.5 3.5) (size 3 3) (drill 1.85) (layers *.Cu *.Mask)
       (net 1 +12V))
+    (model ../../../../../home/cpriscal/Projets/fluffy-potato/edge-connector-motherboard/keystone-PN7770.wrl
+      (at (xyz 0.155 0 -0.2))
+      (scale (xyz 0.393701 0.393701 0.393701))
+      (rotate (xyz -90 0 90))
+    )
   )
   (module edge-connector-motherboard:TERM_SCREW_M3 (layer F.Cu)
@@
     (pad 1 thru_hole circle (at -2.5 3.5) (size 3 3) (drill 1.85) (layers *.Cu *.Mask)
       (net 4 /PIC16F1829LIN/LBUS))
+    (model ../../../../../home/cpriscal/Projets/fluffy-potato/edge-connector-motherboard/keystone-PN7770.wrl
+      (at (xyz 0.155 0 -0.2))
+      (scale (xyz 0.393701 0.393701 0.393701))
+      (rotate (xyz -90 0 90))
+    )
   )
   (module edge-connector-motherboard:TERM_SCREW_M3 (layer F.Cu)
@@
     (pad 1 thru_hole circle (at -2.5 3.5) (size 3 3) (drill 1.85) (layers *.Cu *.Mask)
       (net 26 GNDPWR))
+    (model ../../../../../home/cpriscal/Projets/fluffy-potato/edge-connector-motherboard/keystone-PN7770.wrl
+      (at (xyz 0.155 0 -0.2))
+      (scale (xyz 0.393701 0.393701 0.393701))
+      (rotate (xyz -90 0 90))
+    )
   )
   (module Pin_Headers:Pin_Header_Angled_2x32_Pitch2.54mm (layer F.Cu)
@@
     (pad 64 thru_hole oval (at 2.54 78.74) (size 1.7 1.7) (drill 1) (layers *.Cu *.Mask)
       (net 20 /E8))
-    (model ${KISYS3DMOD}/Pin_Headers.3dshapes/Pin_Header_Angled_2x32_Pitch2.54mm.wrl
-      (at (xyz 0.05 -1.55 0))
-      (scale (xyz 1 1 1))
-      (rotate (xyz 0 0 90))
+    (model ../../../../../home/cpriscal/Projets/fluffy-potato/edge-connector-motherboard/c-1761468-1-b-3d.wrl
+      (at (xyz 0.77 -1.55 0.185))
+      (scale (xyz 0.393701 0.393701 0.393701))
+      (rotate (xyz -90 0 -90))
     )
   )
@@
     (pad 1 thru_hole circle (at -2.5 3.5 90) (size 3 3) (drill 1.85) (layers *.Cu *.Mask)
       (net 6 /E1))
+    (model ../../../../../home/cpriscal/Projets/fluffy-potato/edge-connector-motherboard/keystone-PN7770.wrl
+      (at (xyz 0.155 0 -0.2))
+      (scale (xyz 0.393701 0.393701 0.393701))
+      (rotate (xyz -90 0 90))
+    )
   )
   (module edge-connector-motherboard:TERM_SCREW_M3 (layer F.Cu)
@@
     (pad 1 thru_hole circle (at -2.5 3.5 90) (size 3 3) (drill 1.85) (layers *.Cu *.Mask)
       (net 8 /E2))
+    (model ../../../../../home/cpriscal/Projets/fluffy-potato/edge-connector-motherboard/keystone-PN7770.wrl
+      (at (xyz 0.155 0 -0.2))
+      (scale (xyz 0.393701 0.393701 0.393701))
+      (rotate (xyz -90 0 90))
+    )
   )
   (module edge-connector-motherboard:TERM_SCREW_M3 (layer F.Cu)
@@
     (pad 1 thru_hole circle (at -2.5 3.5 90) (size 3 3) (drill 1.85) (layers *.Cu *.Mask)
       (net 10 /E3))
+    (model ../../../../../home/cpriscal/Projets/fluffy-potato/edge-connector-motherboard/keystone-PN7770.wrl
+      (at (xyz 0.155 0 -0.2))
+      (scale (xyz 0.393701 0.393701 0.393701))
+      (rotate (xyz -90 0 90))
+    )
   )
   (module edge-connector-motherboard:TERM_SCREW_M3 (layer F.Cu)
@@
     (pad 1 thru_hole circle (at -2.5 3.5 90) (size 3 3) (drill 1.85) (layers *.Cu *.Mask)
       (net 12 /E4))
+    (model ../../../../../home/cpriscal/Projets/fluffy-potato/edge-connector-motherboard/keystone-PN7770.wrl
+      (at (xyz 0.155 0 -0.2))
+      (scale (xyz 0.393701 0.393701 0.393701))
+      (rotate (xyz -90 0 90))
+    )
   )
   (module edge-connector-motherboard:TERM_SCREW_M3 (layer F.Cu)
@@
     (pad 1 thru_hole circle (at -2.5 3.5 90) (size 3 3) (drill 1.85) (layers *.Cu *.Mask)
       (net 14 /E5))
+    (model ../../../../../home/cpriscal/Projets/fluffy-potato/edge-connector-motherboard/keystone-PN7770.wrl
+      (at (xyz 0.155 0 -0.2))
+      (scale (xyz 0.393701 0.393701 0.393701))
+      (rotate (xyz -90 0 90))
+    )
   )
   (module edge-connector-motherboard:TERM_SCREW_M3 (layer F.Cu)
@@
     (pad 1 thru_hole circle (at -2.5 3.5 90) (size 3 3) (drill 1.85) (layers *.Cu *.Mask)
       (net 16 /E6))
+    (model ../../../../../home/cpriscal/Projets/fluffy-potato/edge-connector-motherboard/keystone-PN7770.wrl
+      (at (xyz 0.155 0 -0.2))
+      (scale (xyz 0.393701 0.393701 0.393701))
+      (rotate (xyz -90 0 90))
+    )
   )
   (module edge-connector-motherboard:TERM_SCREW_M3 (layer F.Cu)
@@
     (pad 1 thru_hole circle (at -2.5 3.5 90) (size 3 3) (drill 1.85) (layers *.Cu *.Mask)
       (net 18 /E7))
+    (model ../../../../../home/cpriscal/Projets/fluffy-potato/edge-connector-motherboard/keystone-PN7770.wrl
+      (at (xyz 0.155 0 -0.2))
+      (scale (xyz 0.393701 0.393701 0.393701))
+      (rotate (xyz -90 0 90))
+    )
   )
   (module edge-connector-motherboard:TERM_SCREW_M3 (layer F.Cu)
@@
     (pad 1 thru_hole circle (at -2.5 3.5 90) (size 3 3) (drill 1.85) (layers *.Cu *.Mask)
       (net 20 /E8))
+    (model ../../../../../home/cpriscal/Projets/fluffy-potato/edge-connector-motherboard/keystone-PN7770.wrl
+      (at (xyz 0.155 0 -0.2))
+      (scale (xyz 0.393701 0.393701 0.393701))
+      (rotate (xyz -90 0 90))
+    )
   )
   (module Housings_SSOP:SSOP-20_5.3x7.2mm_Pitch0.65mm (layer F.Cu)
@@
   (segment (start 156.21 120.65) (end 156.21 110.49) (width 1.27) (layer B.Cu) (net 2))
   (segment (start 156.21 110.49) (end 156.21 100.33) (width 1.27) (layer B.Cu) (net 2))
+  (segment (start 156.21 100.33) (end 156.21 90.17) (width 1.27) (layer B.Cu) (net 2))
+  (segment (start 156.21 90.17) (end 156.21 80.01) (width 1.27) (layer B.Cu) (net 2))
   (via (at 147.955 143.51) (size 0.508) (layers F.Cu B.Cu) (net 3))
   (via (at 147.955 135.89) (size 0.508) (layers F.Cu B.Cu) (net 3))
@@
   (segment (start 156.21 69.85) (end 156.21 59.69) (width 1.27) (layer B.Cu) (net 26))
   (segment (start 156.21 80.01) (end 156.21 69.85) (width 1.27) (layer B.Cu) (net 26))
-  (segment (start 156.21 90.17) (end 156.21 80.01) (width 1.27) (layer B.Cu) (net 26))
-  (segment (start 156.21 100.33) (end 156.21 90.17) (width 1.27) (layer B.Cu) (net 26))
   (segment (start 153.71 39.06) (end 156.21 39.06) (width 1.27) (layer B.Cu) (net 26))
   (segment (start 156.21 39.06) (end 156.21 49.53) (width 1.27) (layer B.Cu) (net 26))
