File: board_generator/modules/bl652/bl652.kicad_pcb (KiCad board)
At the start: 2 copper layers, 12 parts, among them J1 TEST_1P, J2 TEST_1P, J3 TEST_1P, J4 TEST_1P, U1 BL652, U2 MCP2050, X1 interface, X2 interface

Commit message: bl652 and edge complete
Other:
- board outline added: 22.9 x 20.3 mm
- board text added: "3V3"
- board text added: "GND"
- board text added: "SWDCLK"
- board text added: "SWDIO"
Changed lines of the file:
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@@
     (links 37)
     (no_connects 0)
-    (area 0 0 0 0)
+    (area 122.810199 67.023 170.305801 94.1438)
     (thickness 1.6)
-    (drawings 0)
+    (drawings 7)
     (tracks 196)
     (zones 0)
@@
     (46 B.CrtYd user)
     (47 F.CrtYd user)
-    (48 B.Fab user)
+    (48 B.Fab user hide)
     (49 F.Fab user)
   )
@@
     (pad_drill 0.762)
     (pad_to_mask_clearance 0.2)
-    (aux_axis_origin 0 0)
+    (aux_axis_origin 135.128 90.551)
     (visible_elements FFFFFF7F)
     (pcbplotparams
-      (layerselection 0x00030_80000001)
-      (usegerberextensions false)
+      (layerselection 0x010f0_80000001)
+      (usegerberextensions true)
       (excludeedgelayer true)
       (linewidth 0.100000)
@@
       (viasonmask false)
       (mode 1)
-      (useauxorigin false)
+      (useauxorigin true)
       (hpglpennumber 1)
       (hpglpenspeed 20)
@@
       (outputformat 1)
       (mirror false)
-      (drillshape 1)
+      (drillshape 0)
       (scaleselection 1)
-      (outputdirectory ""))
+      (outputdirectory gbr))
   )
   (net 0 "")
@@
     (tags "capacitor 0805")
     (attr smd)
-    (fp_text reference C1 (at 0 -1.75 180) (layer F.SilkS)
+    (fp_text reference C1 (at -3.429 0 180) (layer F.SilkS)
       (effects (font (size 1 1) (thickness 0.15)))
     )
@@
     (tags "resistor 0603")
     (attr smd)
-    (fp_text reference R1 (at 0 -1.45 180) (layer F.SilkS)
+    (fp_text reference R1 (at -3.429 0 180) (layer F.SilkS)
       (effects (font (size 1 1) (thickness 0.15)))
     )
@@
     (tags "resistor 0603")
     (attr smd)
-    (fp_text reference R2 (at 0 -1.45 180) (layer F.SilkS)
+    (fp_text reference R2 (at -3.472 0 180) (layer F.SilkS)
       (effects (font (size 1 1) (thickness 0.15)))
     )
@@
     (tags "Bluetooth BLE NFC")
     (attr smd)
-    (fp_text reference U1 (at 0 -6.985 270) (layer F.SilkS)
+    (fp_text reference U1 (at 0 0 360) (layer F.SilkS)
       (effects (font (size 1 1) (thickness 0.15)))
     )
@@
     (tags "SOIC 1.27")
     (attr smd)
-    (fp_text reference U2 (at 0 -5.375 180) (layer F.SilkS)
+    (fp_text reference U2 (at 0 0 180) (layer F.SilkS)
       (effects (font (size 1 1) (thickness 0.15)))
     )
@@
     (tags SOD-323)
     (attr smd)
-    (fp_text reference D1 (at 0 -1.85) (layer F.SilkS)
+    (fp_text reference D1 (at 3.429 0) (layer F.SilkS)
       (effects (font (size 1 1) (thickness 0.15)))
     )
@@
     (tags "Mesurement Point Square SMD Pad 1.5x1.5mm")
     (attr virtual)
-    (fp_text reference J1 (at 0 2) (layer B.SilkS)
+    (fp_text reference J1 (at 0 2) (layer B.SilkS) hide
       (effects (font (size 1 1) (thickness 0.15)) (justify mirror))
     )
@@
     (tags "Mesurement Point Square SMD Pad 1.5x1.5mm")
     (attr virtual)
-    (fp_text reference J2 (at 0 2) (layer B.SilkS)
+    (fp_text reference J2 (at 0 2) (layer B.SilkS) hide
       (effects (font (size 1 1) (thickness 0.15)) (justify mirror))
     )
@@
     (tags "Mesurement Point Square SMD Pad 1.5x1.5mm")
     (attr virtual)
-    (fp_text reference J3 (at 0 2) (layer B.SilkS)
+    (fp_text reference J3 (at 0 2) (layer B.SilkS) hide
       (effects (font (size 1 1) (thickness 0.15)) (justify mirror))
     )
@@
     (tags "Mesurement Point Square SMD Pad 1.5x1.5mm")
     (attr virtual)
-    (fp_text reference J4 (at 0 2) (layer B.SilkS)
+    (fp_text reference J4 (at 0 2) (layer B.SilkS) hide
       (effects (font (size 1 1) (thickness 0.15)) (justify mirror))
     )
@@
       (net 2 GND))
   )
+  (dimension 22.86 (width 0.3) (layer Dwgs.User)
+    (gr_text "0.9000 in" (at 146.558 68.373) (layer Dwgs.User)
+      (effects (font (size 1.5 1.5) (thickness 0.3)))
+    )
+    (feature1 (pts (xy 157.988 72.136) (xy 157.988 67.023)))
+    (feature2 (pts (xy 135.128 72.136) (xy 135.128 67.023)))
+    (crossbar (pts (xy 135.128 69.723) (xy 157.988 69.723)))
+    (arrow1a (pts (xy 157.988 69.723) (xy 156.861496 70.309421)))
+    (arrow1b (pts (xy 157.988 69.723) (xy 156.861496 69.136579)))
+    (arrow2a (pts (xy 135.128 69.723) (xy 136.254504 70.309421)))
+    (arrow2b (pts (xy 135.128 69.723) (xy 136.254504 69.136579)))
+  )
+  (gr_text SWDCLK (at 155.956 82.55 90) (layer B.SilkS)
+    (effects (font (size 1.5 1.5) (thickness 0.3)) (justify left mirror))
+  )
+  (gr_text SWDIO (at 153.67 82.423 90) (layer B.SilkS)
+    (effects (font (size 1.5 1.5) (thickness 0.3)) (justify left mirror))
+  )
+  (gr_text 3V3 (at 151.13 82.55 90) (layer B.SilkS)
+    (effects (font (size 1.5 1.5) (thickness 0.3)) (justify left mirror))
+  )
+  (gr_text GND (at 148.717 82.55 90) (layer B.SilkS)
+    (effects (font (size 1.5 1.5) (thickness 0.3)) (justify left mirror))
+  )
+  (gr_line (start 135.128 92.456) (end 157.988 92.456) (layer Edge.Cuts) (width 0.15))
+  (gr_line (start 157.988 72.136) (end 135.128 72.136) (layer Edge.Cuts) (width 0.15))
   (via (at 143.679657 84.963) (size 0.762) (drill 0.381) (layers F.Cu B.Cu) (net 1))
   (segment (start 148.971 84.963) (end 143.679657 84.963) (width 0.508) (layer B.Cu) (net 1))
